File: esp32-laser-security-pcb/_restore_backup_2026-06-05T10-23-50-833/esp32-laser-security.kicad_pcb (KiCad board)
At the start: 2 copper layers, 46.5 x 37.5 mm, 9 parts, among them J1 Conn_01x06, SW1 SW_Push

Commit message: Updated pcb design and add schematic and 3D PCB render images for laser security board
Parts:
- removed REF** (x4): MountingHole_3.2mm_M3, MountingHole:MountingHole_3.2mm_M3
- moved J1 2.36 mm to (93.5, 88.7)
Routing:
- net Net-(J1-Pin_6): track 68.3 -> 35.8 mm
- net Net-(BZ1-+): track 47.7 -> 35.1 mm
- net Net-(BZ1--): track 60.6 -> 71.2 mm
- net Net-(J1-Pin_5): track 42.1 -> 33.6 mm
- net Net-(J1-Pin_1): track 11.6 -> 10.1 mm
Other:
- board outline removed
- board text removed: "Jaswant Bh."
