File: pcb/esp32-laser-security.kicad_sch (KiCad schematic)
At the start: 5 parts, among them J1 Conn_01x06, SW1 SW_Push

Commit message: Updated pcb design and add schematic and 3D PCB render images for laser security board
Parts:
- SW1: footprint Button_Switch_THT:SW_PUSH_6mm -> (none)
Changed lines of the file:
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@@
 			)
 		)
-		(property "Footprint" "Button_Switch_THT:SW_PUSH_6mm"
+		(property "Footprint" ""
 			(at 208.28 63.5 0)
 			(hide yes)
